File: jorian.kicad_pcb (KiCad board)
At the start: 2 copper layers, 98.9 x 100 mm, 90 parts, among them J6 lipo_charger, U3 LP3990-3.3v

Commit message: first commit
Parts:
- removed G1, G2: Logo_Open_Hardware_Small, kbd:jorian_logo
- removed J6: lipo_charger, kbd:lipo_charger_03962A
- removed JP11, JP22: VUSB, kbd:jumper
- removed JP12, JP23: GND, kbd:jumper
- removed JP13, JP24: OUT+, kbd:jumper
- removed JP14, JP25: LIPO+, kbd:jumper
- removed JP15, JP26: LIPO-, kbd:jumper
- removed JP17, JP27: OUT-, kbd:jumper
- removed U2: ~, kbd:nrf51822_smd
- U1: value ~ -> E73-2G4M08S1C-52840; footprint kbd:nrf51822_smd -> kbd:E73-2G4M08S1C-52840
- moved U1 8.13 mm to (88.1, 98.4)
Connections:
- U1 pad 1: GND -> Net-(U1-Pad1)
- U1 pad 10: /S10 -> Net-(U1-Pad10)
- U1 pad 11: GND -> Net-(U1-Pad11)
- U1 pad 12: VCC -> Net-(U1-Pad12)
- U1 pad 13: /S3 -> Net-(U1-Pad13)
- U1 pad 14: /S14 -> Net-(U1-Pad14)
- U1 pad 15: /S9 -> Net-(U1-Pad15)
- U1 pad 16: /S8 -> Net-(U1-Pad16)
- U1 pad 17: /S13 -> Net-(U1-Pad17)
- U1 pad 18: /S2 -> Net-(U1-Pad18)
- U1 pad 19: /S7 -> Net-(U1-Pad19)
- U1 pad 2: /S15 -> Net-(U1-Pad2)
- U1 pad 20: /S12 -> Net-(U1-Pad20)
- U1 pad 21: /S1 -> Net-(U1-Pad21)
- U1 pad 22: /S6 -> Net-(U1-Pad22)
- U1 pad 23: /S11 -> Net-(U1-Pad23)
- U1 pad 24: /S19 -> Net-(U1-Pad24)
- U1 pad 25: SDA -> Net-(U1-Pad25)
- U1 pad 26: SCL -> Net-(U1-Pad26)
- U1 pad 27: /S17 -> Net-(U1-Pad27)
- U1 pad 28: /S18 -> Net-(U1-Pad28)
- U1 pad 29: /S20 -> Net-(U1-Pad29)
- U1 pad 3: TX -> Net-(U1-Pad3)
- U1 pad 30: /S16 -> Net-(U1-Pad30)
- U1 pad 31: SWD -> Net-(U1-Pad31)
- U1 pad 32: SWC -> Net-(U1-Pad32)
- U1 pad 33: /S21 -> Net-(U1-Pad33)
- U1 pad 34: /S22 -> Net-(U1-Pad34)
- U1 pad 35: LED_DATA -> Net-(U1-Pad35)
- U1 pad 36: SWO -> Net-(U1-Pad36)
- U1 pad 4: /LED -> Net-(U1-Pad4)
- U1 pad 5: /S4 -> Net-(U1-Pad5)
- U1 pad 6: RX -> Net-(U1-Pad6)
- U1 pad 9: /S5 -> Net-(U1-Pad9)
Routing:
- net GND: track 995.1 -> 0.00 mm, vias 5 -> 0
- net VCC: track 636.3 -> 0.00 mm, vias 23 -> 0
- net /GND_B: track 244.3 -> 0.00 mm, vias 4 -> 0
- net /VCC_B: track 122.5 -> 0.00 mm, vias 7 -> 0
- net /S20: track 120.6 -> 0.00 mm, vias 5 -> 0
- net /S4: track 118.2 -> 0.00 mm, vias 11 -> 0
- net /S19: track 105.8 -> 0.00 mm, vias 5 -> 0
- net /S1: track 100.4 -> 0.00 mm, vias 3 -> 0
- net BAT-: track 100.2 -> 0.00 mm, vias 4 -> 0
- net /S20_B: track 99.3 -> 0.00 mm, vias 6 -> 0
- net /S22: track 92.6 -> 0.00 mm, vias 5 -> 0
- net /S15: track 86.3 -> 0.00 mm, vias 5 -> 0
- net /S21: track 85.9 -> 0.00 mm, vias 1 -> 0
- net /S5: track 85.7 -> 0.00 mm, vias 4 -> 0
- net OUT+: track 84.2 -> 0.00 mm, vias 6 -> 0
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
Commit message: updated
Parts:
- OLED1: footprint kbd:connector_i2c -> kbd:oled_128x32_i2c; moved to F.Cu
- moved JP3 18.3 mm to (78.4, 107.3)
- moved JP7 18.3 mm to (78.4, 107.3)
- moved JP2 18.3 mm to (78.4, 109.9)
- moved JP4 18.3 mm to (78.4, 104.8)
- moved JP5 18.3 mm to (78.4, 102.2)
- moved JP6 18.3 mm to (78.4, 109.9)
- moved JP8 18.3 mm to (78.4, 104.8)
- moved JP9 18.3 mm to (78.4, 102.2)
- moved JP1 11.0 mm to (78.1, 99.7)
- moved JP10 11.0 mm to (78.1, 99.7)
- moved OLED1 6.59 mm to (80.6, 106.0), turned to 90 degrees
- moved H1 2.21 mm to (90.2, 104.8)
- moved U1 0.80 mm to (88.9, 98.4)
- moved BT1 0.42 mm to (90.8, 109.9)
- moved L17 0.07 mm to (69.8, 104.8)
Other:
- outline, holes or cut-outs redrawn

Commit message: updated files
Parts:
- added C3: 10uF, Capacitor_SMD:C_0805_2012Metric, F.Cu at (79.4, 59.7)
- added D1: CHG, LED_SMD:LED_0603_1608Metric, B.Cu at (43.2, 49.7)
- added D2: 1N5819, Diode_SMD:D_SOD-323, F.Cu at (79.4, 42.5)
- added J1: MicroUSB, kbd:usb_micro_custom, F.Cu at (51.4, 38.7)
- added J2: MicroUSB, kbd:usb_micro_custom, B.Cu at (51.4, 38.7)
- added J3: USB-C, kbd:usb_type_c, B.Cu at (51.4, 38.7)
- added J4: USB-C, kbd:usb_type_c, F.Cu at (51.4, 38.7)
- added J5: MJ-4PP-9, kbd:trrs_connector, F.Cu at (43.2, 64.1)
- added JP11: SWD_conn, kbd:connector_swd, F.Cu at (73.0, 40.6)
- added JP12: TX, kbd:jumper, F.Cu at (76.8, 42.5)
- added JP13: RX, kbd:jumper, F.Cu at (59.1, 42.5)
- added JP14: VCC, kbd:jumper, F.Cu at (69.2, 42.5)
- added JP15: GND, kbd:jumper, F.Cu at (74.3, 42.5)
- added JP17: VCC, kbd:jumper, F.Cu at (61.6, 42.5)
- added JP22: GND, kbd:jumper, F.Cu at (66.7, 42.5)
- added JP23: D+, kbd:jumper, F.Cu at (64.1, 42.5)
- added JP24: D-, kbd:jumper, F.Cu at (71.8, 42.5)
- added Q1: AO3407, Package_TO_SOT_SMD:SOT-23, F.Cu at (79.4, 53.3)
- added R1: 5.1K, Resistor_SMD:R_0603_1608Metric, F.Cu at (60.5, 47.6)
- added R2: 5.1K, Resistor_SMD:R_0603_1608Metric, F.Cu at (60.3, 49.5)
- added R3: 1.5K, kbd:R_0805, F.Cu at (60.3, 57.1)
- added R4: 1.5K, kbd:R_0805, F.Cu at (60.3, 60.3)
- added R5: 100K, Resistor_SMD:R_0603_1608Metric, F.Cu at (79.4, 65.4)
- added R6: 1K, Resistor_SMD:R_0603_1608Metric, F.Cu at (43.2, 49.7)
- added R7: 10K, Resistor_SMD:R_0603_1608Metric, F.Cu at (60.3, 51.4)
- added R8: 100K, Resistor_SMD:R_0603_1608Metric, F.Cu at (79.4, 61.6)
- added R9: 4.7K, Resistor_SMD:R_0603_1608Metric, F.Cu at (79.4, 63.5)
- added SW1: MSK-12C02, kbd:switch_MSK-12C02_smd, F.Cu at (41.9, 43.2)
- added U2: MCP73831, Package_TO_SOT_SMD:SOT-23-5, F.Cu at (79.4, 46.4)
- C1, C2: value 1uF -> 10uF; footprint kbd:C_0805 -> Capacitor_SMD:C_0805_2012Metric
- U3: value LP3990-3.3v -> AP2112K-3.3; footprint kbd:SOT-23-5 -> Package_TO_SOT_SMD:SOT-23-5
- moved U3 50.4 mm to (79.4, 50.2), turned to 0 degrees
- moved C1 44.3 mm to (79.4, 55.9), turned to 0 degrees
- moved C2 43.8 mm to (79.4, 57.8), turned to 0 degrees
Connections:
- C1 pad 1: OUT+ -> Net-(C1-Pad1)
- C2 pad 1: VCC -> VBAT
- U3 pad 1: OUT+ -> Net-(C1-Pad1)
- U3 pad 3: OUT+ -> Net-(R8-Pad2)

Commit message: updated files
Parts:
- added JP25: , kbd:jumper, B.Cu at (64.1, 42.5)
- added JP26: , kbd:jumper, B.Cu at (61.6, 42.5)
- added JP27: , kbd:jumper, B.Cu at (59.1, 42.5)
- added JP28: , kbd:jumper, F.Cu at (66.7, 42.5)
- added JP29: , kbd:jumper, F.Cu at (64.1, 42.5)
- added JP30: , kbd:jumper, F.Cu at (61.6, 42.5)
- added JP31: , kbd:jumper, F.Cu at (59.1, 42.5)
- added OLED2: I2C_conn, kbd:connector_i2c, F.Cu at (62.9, 40.6)
- JP16: value SWD_conn -> (none); footprint kbd:connector_swd -> kbd:jumper; moved to B.Cu
- JP22, JP23: moved to B.Cu
- OLED1: footprint kbd:oled_128x32_i2c -> kbd:connector_i2c
- moved JP16 69.5 mm to (66.7, 42.5)
- moved JP22 24.8 mm to (57.1, 65.4)
- moved JP17 23.3 mm to (57.1, 65.4)
- moved JP23 21.6 mm to (57.1, 63.0)
- moved JP13 20.5 mm to (57.1, 63.0)
- moved U3 19.4 mm to (60.3, 54.0)
- moved Q1 19.3 mm to (60.3, 50.2)
- moved U2 19.0 mm to (60.3, 46.4)
- moved R7 17.2 mm to (43.2, 52.7), turned to 270 degrees
- moved JP1 14.0 mm to (64.1, 99.7)
- moved R1 11.8 mm to (51.4, 40.0)
- moved R2 11.7 mm to (51.4, 41.9)
- moved C1 10.2 mm to (79.4, 45.7)
- moved C2 9.52 mm to (79.4, 48.3)
- moved C3 8.89 mm to (79.4, 50.8)
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Connections:
- JP16 pad 1: VCC -> GND
- JP16 pad 2: GND -> Net-(JP16-Pad2)

Commit message: updated files
Parts:
- removed JP12: TX, kbd:jumper
- removed JP13: RX, kbd:jumper
- removed JP14, JP17: VCC, kbd:jumper
- removed JP15, JP22: GND, kbd:jumper
- removed JP23: D+, kbd:jumper
- removed JP24: D-, kbd:jumper
- removed R3, R4: 1.5K, kbd:R_0805
- C1, C2, C3: footprint Capacitor_SMD:C_0805_2012Metric -> Capacitor_SMD:C_0603_1608Metric
- D2: footprint Diode_SMD:D_SOD-323 -> Diode_SMD:D_SOD-123
- moved JP1 25.6 mm to (89.5, 103.0)
- moved D2 25.2 mm to (60.3, 59.1)
- moved JP10 20.0 mm to (89.5, 103.0)
- moved JP18 3.18 mm to (72.4, 99.8)
- moved JP19 3.18 mm to (72.4, 99.8)
- moved JP20 3.18 mm to (67.3, 99.8)
- moved JP21 3.18 mm to (67.3, 99.8)
- moved H1 2.62 mm to (89.5, 107.3)
- moved SW1 0.18 mm to (41.9, 43.0)
Connections:
- J5 pad B: Net-(J5-PadB) -> RX
- J5 pad C: Net-(J5-PadC) -> GND
- J5 pad D: Net-(J5-PadD) -> VCC

Commit message: updated files
Parts:
- added U4: E73-2G4M08S1C-52840, kbd:E73-2G4M08S1C-52840-mod, B.Cu at (88.9, 98.4)
- U1: footprint kbd:E73-2G4M08S1C-52840 -> kbd:E73-2G4M08S1C-52840-mod
- moved R7 32.8 mm to (74.8, 43.8), turned to 0 degrees
- moved R6 28.7 mm to (71.3, 43.8), turned to 0 degrees
- moved D2 10.0 mm to (69.8, 62.2), turned to 0 degrees
- moved U3 6.35 mm to (60.3, 60.3)
- moved R5 4.45 mm to (79.4, 61.6)
- moved Q1 3.81 mm to (60.3, 54.0)
- moved R9 3.81 mm to (79.4, 59.1)
- moved R8 2.54 mm to (79.4, 55.9)
- moved C3 1.91 mm to (79.4, 52.7)
- moved U2 1.91 mm to (60.3, 48.3)
- moved C2 1.27 mm to (79.4, 49.5)
- moved C1 0.63 mm to (79.4, 46.4)
- moved H1 0.63 mm to (88.9, 107.3)
- moved JP1 0.63 mm to (88.9, 103.0)
- moved JP10 0.63 mm to (88.9, 103.0)

Commit message: latest changes
Parts:
- D1: moved to F.Cu
- R6, R7: moved to B.Cu
- moved R2 25.5 mm to (76.8, 43.8)
- moved R1 20.7 mm to (71.8, 43.8)
- moved JP20 18.7 mm to (78.4, 114.9), turned to 90 degrees
- moved JP21 18.7 mm to (78.4, 114.9), turned to 90 degrees
- moved JP18 13.9 mm to (78.4, 112.4), turned to 270 degrees
- moved JP19 13.9 mm to (78.4, 112.4), turned to 90 degrees
- moved R7 2.06 mm to (76.8, 43.8), turned to 180 degrees
- moved D1 1.14 mm to (42.3, 50.4), turned to 90 degrees
- moved JP16 0.90 mm to (67.3, 43.2)
- moved JP28 0.90 mm to (67.3, 43.2)
- moved JP26 0.90 mm to (62.2, 43.2)
- moved JP27 0.90 mm to (59.7, 43.2)
- moved JP30 0.90 mm to (62.2, 43.2)
- moved JP31 0.90 mm to (59.7, 43.2)
- moved JP25 0.90 mm to (64.8, 43.2)
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
Commit message: updated files
Parts:
- J3, J4: footprint kbd:usb_type_c -> kbd:HRO-TYPE-C-31-M-12-Assembly
- S1, S10, S11, S12, S13, S14, S15, S16, S17, S18, S19, S2, S20, S21, S22, S3, S4, S5, S6, S7, S8, S9: footprint kbd:cherry -> kbd:universal_footprint_cutouts
- moved D2 11.4 mm to (60.3, 56.0), turned to 90 degrees
- moved Q1 2.54 mm to (60.3, 51.4)
- moved U2 1.91 mm to (60.3, 46.4)
- moved U3 0.28 mm to (60.2, 60.6)
- turned J3 to 0 degrees
- turned J4 to 180 degrees
