File: jorian.kicad_pcb (KiCad board)
At the start: 2 copper layers, 98.9 x 100 mm, 102 parts, among them J1 MicroUSB, J2 MicroUSB, J3 USB-C, J4 USB-C, J5 MJ-4PP-9, Q1 AO3407, SW1 MSK-12C02, U1 E73-2G4M08S1C-52840, U2 MCP73831, U3 AP2112K-3.3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

Commit message: updated files
Parts:
- removed R8: 100K, Resistor_SMD:R_0603_1608Metric
- removed the U3 at (60.2, 60.6)
- added X1: 10uH, Inductor_SMD:L_0603_1608Metric, F.Cu at (87.1, 95.0)
- J1: renamed from J4; footprint kbd:HRO-TYPE-C-31-M-12-Assembly -> kbd:usb_type_c
- J2: renamed from J3; footprint kbd:HRO-TYPE-C-31-M-12-Assembly -> kbd:usb_type_c
- S1, S10, S11, S12, S13, S14, S15, S16, S17, S18, S19, S2, S20, S21, S22, S3, S4, S5, S6, S7, S8, S9: footprint kbd:universal_footprint_cutouts -> kbd:cherry
- U1: footprint kbd:E73-2G4M08S1C-52840-mod -> kbd:E73-2G4M08S1C-52840
- U2: renamed from U4; footprint kbd:E73-2G4M08S1C-52840-mod -> kbd:E73-2G4M08S1C-52840
- moved D1 28.9 mm to (70.4, 43.4), turned to 0 degrees
- moved R5 23.5 mm to (61.3, 46.5), turned to 270 degrees
- moved R2 19.6 mm to (57.3, 45.6), turned to 90 degrees
- moved R7 19.6 mm to (57.3, 45.6), turned to 270 degrees
- moved Q1 19.3 mm to (79.4, 48.1), turned to 270 degrees
- moved U3 19.3 mm to (79.5, 44.2)
- moved D2 18.9 mm to (74.5, 43.6), turned to 0 degrees
- moved C2 18.1 mm to (61.3, 51.5), turned to 90 degrees
- moved R9 18.1 mm to (61.3, 57.9), turned to 270 degrees
- moved R1 14.9 mm to (57.3, 40.5), turned to 90 degrees
- moved R6 14.9 mm to (57.3, 40.5), turned to 270 degrees
- moved C1 11.6 mm to (78.5, 57.9), turned to 90 degrees
- moved JP1 8.60 mm to (89.5, 94.9)
- moved JP10 8.60 mm to (89.5, 94.9)
- moved C3 1.45 mm to (78.5, 51.6), turned to 90 degrees
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- renumbered J1 to J3, J2 to J4, U2 to U3
Connections:
- net P0.26 renamed P0.05
- C1 pad 1: Net-(C1-Pad1) -> VDDH
- C3 pad 1: VCC -> VDDH
- D2 pad 1: Net-(C1-Pad1) -> VDDH
- E10 pad 2: /S22 -> S22
- E15 pad 2: /S21 -> S21
- E16 pad 2: /S18 -> S18
- E5 pad 2: /S19 -> S19
- E5 pad 3: /S20 -> S20
- Q1 pad 2: Net-(C1-Pad1) -> VDDH
- R1 pad 1: Net-(J3-PadA5) -> Net-(J2-PadA5)
- R2 pad 1: Net-(J3-PadB5) -> Net-(J2-PadB5)
- S1 pad 2: /S1 -> S1
- S10 pad 2: /S10 -> S10
- S11 pad 2: /S11 -> S11
- S12 pad 2: /S12 -> S12
- S13 pad 2: /S13 -> S13
- S14 pad 2: /S14 -> S14
- S15 pad 2: /S15 -> S15
- S16 pad 2: /S16 -> S16
- S17 pad 2: /S17 -> S17
- S2 pad 2: /S2 -> S2
- S3 pad 2: /S3 -> S3
- S4 pad 2: /S4 -> S4
- S5 pad 2: /S5 -> S5
- S6 pad 2: /S6 -> S6
- S7 pad 2: /S7 -> S7
- S8 pad 2: /S8 -> S8
- S9 pad 2: /S9 -> S9
- U1 pad 1: Net-(U1-Pad1) -> S1
- U1 pad 10: Net-(U1-Pad10) -> S9
- U1 pad 11: Net-(U1-Pad11) -> SDA
- U1 pad 13: Net-(U1-Pad13) -> SCL
- U1 pad 15: Net-(U1-Pad15) -> S10
- U1 pad 17: Net-(U1-Pad17) -> S11
- U1 pad 19: Net-(U1-Pad19) -> VDD
- U1 pad 2: Net-(U1-Pad2) -> S2
- U1 pad 21: Net-(U1-Pad21) -> GND
- U1 pad 23: Net-(U1-Pad23) -> VDDH
- U1 pad 25: Net-(U1-Pad25) -> DCCH
- U1 pad 26: Net-(U1-Pad26) -> RESET
- U1 pad 27: Net-(U1-Pad27) -> VBUS
- U1 pad 28: Net-(U1-Pad28) -> POWER_PIN
- U1 pad 29: Net-(U1-Pad29) -> D-
- U1 pad 3: Net-(U1-Pad3) -> S3
- U1 pad 30: Net-(U1-Pad30) -> S22
- U1 pad 31: Net-(U1-Pad31) -> D+
- U1 pad 32: Net-(U1-Pad32) -> S21
- U1 pad 33: Net-(U1-Pad33) -> S20
- U1 pad 34: Net-(U1-Pad34) -> S19
- U1 pad 35: Net-(U1-Pad35) -> S18
- U1 pad 36: Net-(U1-Pad36) -> S17
- U1 pad 37: Net-(U1-Pad37) -> SWD
- U1 pad 38: Net-(U1-Pad38) -> S16
- U1 pad 39: Net-(U1-Pad39) -> SWC
- U1 pad 4: Net-(U1-Pad4) -> S4
- U1 pad 40: Net-(U1-Pad40) -> S15
- U1 pad 41: Net-(U1-Pad41) -> S14
- U1 pad 42: Net-(U1-Pad42) -> S13
- U1 pad 43: Net-(U1-Pad43) -> S12
- U1 pad 5: Net-(U1-Pad5) -> GND
- U1 pad 6: Net-(U1-Pad6) -> S5
- U1 pad 7: Net-(U1-Pad7) -> S6
- U1 pad 8: Net-(U1-Pad8) -> S7
- U1 pad 9: Net-(U1-Pad9) -> S8
- U2 pad 1: Net-(U4-Pad1) -> S1
- U2 pad 10: Net-(U4-Pad10) -> S9
- U2 pad 11: Net-(U4-Pad11) -> SDA
- U2 pad 13: Net-(U4-Pad13) -> SCL
- U2 pad 15: Net-(U4-Pad15) -> S10
- U2 pad 17: Net-(U4-Pad17) -> S11
- U2 pad 19: Net-(U4-Pad19) -> VDD
- U2 pad 2: Net-(U4-Pad2) -> S2
- U2 pad 21: Net-(U4-Pad21) -> GND
- U2 pad 23: Net-(U4-Pad23) -> VDDH
- U2 pad 25: Net-(U4-Pad25) -> DCCH
- U2 pad 26: Net-(U4-Pad26) -> RESET
- U2 pad 27: Net-(U4-Pad27) -> VBUS
- U2 pad 28: Net-(U4-Pad28) -> POWER_PIN
- U2 pad 29: Net-(U4-Pad29) -> D-
- U2 pad 3: Net-(U4-Pad3) -> S3
- U2 pad 30: Net-(U4-Pad30) -> S22
- U2 pad 31: Net-(U4-Pad31) -> D+
- U2 pad 32: Net-(U4-Pad32) -> S21
- U2 pad 33: Net-(U4-Pad33) -> S20
- U2 pad 34: Net-(U4-Pad34) -> S19
- U2 pad 35: Net-(U4-Pad35) -> S18
- U2 pad 36: Net-(U4-Pad36) -> S17
- U2 pad 37: Net-(U4-Pad37) -> SWD
- U2 pad 38: Net-(U4-Pad38) -> S16
- U2 pad 39: Net-(U4-Pad39) -> SWC
- U2 pad 4: Net-(U4-Pad4) -> S4
- U2 pad 40: Net-(U4-Pad40) -> S15
- U2 pad 41: Net-(U4-Pad41) -> S14
- U2 pad 42: Net-(U4-Pad42) -> S13
- U2 pad 43: Net-(U4-Pad43) -> S12
- U2 pad 5: Net-(U4-Pad5) -> GND
- U2 pad 6: Net-(U4-Pad6) -> S5
- U2 pad 7: Net-(U4-Pad7) -> S6
- U2 pad 8: Net-(U4-Pad8) -> S7
- U2 pad 9: Net-(U4-Pad9) -> S8

Commit message: updated files
Parts:
- OLED1: footprint kbd:connector_i2c -> kbd:connector_swd
- S10, S15, S19, S20, S21, S5: moved to B.Cu
- turned S10 to 180 degrees
- turned S15 to 180 degrees
- turned S19 to 270 degrees
- turned S20 to 270 degrees
- turned S21 to 270 degrees
- turned S5 to 180 degrees
Connections:
- net BLUE_LED renamed P0.06
- E10 pad 1: GND -> Net-(E10-Pad1)
- E10 pad 3: Net-(E10-Pad3) -> GND
- E10 pad 4: VCC -> S20
- E15 pad 1: GND -> Net-(E15-Pad1)
- E15 pad 2: S21 -> VCC
- E15 pad 3: /DIN21 -> GND
- E15 pad 4: VCC -> S21
- E16 pad 1: GND -> VCC
- E16 pad 2: S18 -> /DIN18
- E16 pad 3: /DIN18 -> GND
- E16 pad 4: VCC -> S18
- E18 pad 1: /GND_A -> /VCC_A
- E18 pad 2: /S18_A -> /DIN18_A
- E18 pad 3: /DIN18_A -> /GND_A
- E18 pad 4: /VCC_A -> /S18_A
- E19 pad 1: /GND_B -> /DIN5_B
- E19 pad 2: /S19_B -> /DIN21_B
- E19 pad 3: /S20_B -> /GND_B
- E19 pad 4: /DIN5_B -> /S19_B
- E20 pad 1: /GND_B -> Net-(E20-Pad1)
- E20 pad 3: Net-(E20-Pad3) -> /GND_B
- E20 pad 4: /VCC_B -> /S20_B
- E21 pad 1: /GND_B -> Net-(E21-Pad1)
- E21 pad 2: /S21_B -> /VCC_B
- E21 pad 3: /DIN21_B -> /GND_B
- E21 pad 4: /VCC_B -> /S21_B
- E5 pad 1: GND -> /DIN5
- E5 pad 2: S19 -> /DIN21
- E5 pad 3: S20 -> GND
- E5 pad 4: /DIN5 -> S19
- U1 pad 28: POWER_PIN -> RX
- U2 pad 28: POWER_PIN -> RX

Commit message: updated files
Parts:
- removed H1: Battery Pad, kbd:battery_pad
- removed JP1: +, kbd:jumper
- removed JP10: -, kbd:jumper
- removed JP16, JP25, JP26, JP27, JP28, JP29, JP30, JP31: , kbd:jumper
- removed OLED2: I2C_conn, kbd:connector_i2c
- added Q2: SI2306, Package_TO_SOT_SMD:SOT-23, F.Cu at (76.8, 41.9)
- added R3: 10K, Resistor_SMD:R_0603_1608Metric, F.Cu at (79.4, 43.3)
- JP19: moved to B.Cu
- JP20, R6, R7: moved to F.Cu
- moved JP11 73.4 mm to (80.6, 113.7), turned to 90 degrees
- moved JP20 55.2 mm to (90.5, 40.0), turned to 90 degrees
- moved JP19 55.2 mm to (87.5, 40.0), turned to 90 degrees
- moved JP18 55.0 mm to (87.5, 40.0), turned to 270 degrees
- moved JP21 55.0 mm to (90.5, 40.0), turned to 270 degrees
- moved X1 54.9 mm to (79.4, 40.6), turned to 270 degrees
- moved C1 22.5 mm to (64.1, 40.6), turned to 270 degrees
- moved R9 19.5 mm to (74.3, 43.3), turned to 90 degrees
- moved C2 16.9 mm to (74.3, 40.6), turned to 270 degrees
- moved C3 14.3 mm to (69.2, 40.6), turned to 270 degrees
- moved Q1 14.1 mm to (66.7, 41.9), turned to 0 degrees
- moved D2 12.4 mm to (62.2, 41.9), turned to 90 degrees
- moved R7 12.2 mm to (69.2, 43.2), turned to 90 degrees
- moved D1 11.0 mm to (59.7, 40.6), turned to 90 degrees
- moved U3 8.08 mm to (71.8, 41.9), turned to 180 degrees
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
Commit message: updated files
Parts:
- moved JP19 20.9 mm to (66.6, 39.9)
- moved JP18 20.9 mm to (66.6, 39.9)
- moved JP20 18.5 mm to (72.0, 39.9)
- moved JP21 18.5 mm to (72.0, 39.9)
- moved Q1 0.89 mm to (66.7, 42.8)
- moved U3 0.89 mm to (71.8, 42.8)
- moved JP11 0.25 mm to (80.4, 113.7)
- moved OLED1 0.25 mm to (80.4, 106.0)
- moved U1 0.13 mm to (88.4, 98.7)
- moved U2 0.08 mm to (88.4, 98.7)

Commit message: updated files
Parts:
- removed J3, J4: MicroUSB, kbd:usb_micro_custom
- moved JP21 15.6 mm to (62.0, 51.8), turned to 180 degrees
- moved JP20 15.6 mm to (62.0, 51.8), turned to 0 degrees
- moved JP18 8.14 mm to (62.0, 46.6), turned to 180 degrees
- moved JP19 8.13 mm to (62.0, 46.6), turned to 0 degrees
- moved Q1 0.77 mm to (66.8, 42.0)
- moved U3 0.76 mm to (71.8, 42.0)

Commit message: updated files
Parts:
- removed JP18: LIPO+, kbd:jumper
- removed JP19: LIPO-, kbd:jumper
- removed JP20: BAT+, kbd:jumper
- removed JP21: BAT-, kbd:jumper
- added Q3: AO3407, Package_TO_SOT_SMD:SOT-23, F.Cu at (77.5, 43.2)
- moved R3 9.86 mm to (69.8, 40.8), turned to 0 degrees
- moved R7 8.57 mm to (77.5, 40.9), turned to 0 degrees
- moved C2 4.59 mm to (69.8, 39.5), turned to 0 degrees
- moved C3 4.59 mm to (73.7, 39.5), turned to 0 degrees
- moved R6 3.50 mm to (62.1, 40.8), turned to 180 degrees
- moved Q2 3.42 mm to (73.7, 43.2), turned to 90 degrees
- moved R5 3.00 mm to (65.9, 40.9), turned to 0 degrees
- moved D1 2.65 mm to (62.1, 39.5), turned to 0 degrees
- moved R9 2.64 mm to (73.7, 40.8), turned to 180 degrees
- moved X1 2.29 mm to (77.5, 39.4), turned to 0 degrees
- moved U3 2.22 mm to (69.8, 43.2), turned to 270 degrees
- moved C1 2.09 mm to (65.9, 39.5), turned to 180 degrees
- moved D2 1.40 mm to (62.2, 43.3), turned to 0 degrees
- moved Q1 1.37 mm to (66.0, 43.2), turned to 90 degrees
- moved U1 0.78 mm to (89.1, 98.5)
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Connections:
- C1 pad 2: GND -> BAT-
- C2 pad 1: VBAT -> BAT+
- C2 pad 2: GND -> BAT-
- C3 pad 1: VDDH -> VDD
- C3 pad 2: GND -> BAT-
- E10 pad 3: GND -> BAT-
- E15 pad 2: VCC -> LED_VCC
- E15 pad 3: GND -> BAT-
- E16 pad 1: VCC -> LED_VCC
- E16 pad 3: GND -> BAT-
- E5 pad 3: GND -> BAT-
- J1 pad A1: GND -> BAT-
- J1 pad A12: GND -> BAT-
- J1 pad B1: GND -> BAT-
- J1 pad B12: GND -> BAT-
- J2 pad A1: GND -> BAT-
- J2 pad A12: GND -> BAT-
- J2 pad B1: GND -> BAT-
- J2 pad B12: GND -> BAT-
- J5 pad C: GND -> BAT-
- J5 pad D: VCC -> VDD
- JP2 pad 1: GND -> BAT-
- JP3 pad 1: VCC -> VDD
- JP8 pad 1: VCC -> VDD
- JP9 pad 1: GND -> BAT-
- L1 pad 2: GND -> BAT-
- L1 pad 4: VCC -> LED_VCC
- L10 pad 2: GND -> BAT-
- L10 pad 4: VCC -> LED_VCC
- L11 pad 2: GND -> BAT-
- L11 pad 4: VCC -> LED_VCC
- L12 pad 2: GND -> BAT-
- L12 pad 4: VCC -> LED_VCC
- L13 pad 2: GND -> BAT-
- L13 pad 4: VCC -> LED_VCC
- L14 pad 2: GND -> BAT-
- L14 pad 4: VCC -> LED_VCC
- L15 pad 2: GND -> BAT-
- L15 pad 4: VCC -> LED_VCC
- L16 pad 2: GND -> BAT-
- L16 pad 4: VCC -> LED_VCC
- L17 pad 2: GND -> BAT-
- L17 pad 4: VCC -> LED_VCC
- L2 pad 2: GND -> BAT-
- L2 pad 4: VCC -> LED_VCC
- L3 pad 2: GND -> BAT-
- L3 pad 4: VCC -> LED_VCC
- L4 pad 2: GND -> BAT-
- L4 pad 4: VCC -> LED_VCC
- L5 pad 2: GND -> BAT-
- L5 pad 4: VCC -> LED_VCC
- L6 pad 2: GND -> BAT-
- L6 pad 4: VCC -> LED_VCC
- L7 pad 2: GND -> BAT-
- L7 pad 4: VCC -> LED_VCC
- L8 pad 2: GND -> BAT-
- L8 pad 4: VCC -> LED_VCC
- L9 pad 2: GND -> BAT-
- L9 pad 4: VCC -> LED_VCC
- Q2 pad 2: GND -> BAT-
- Q2 pad 3: LED_GND -> Net-(Q2-Pad3)
- R1 pad 2: GND -> BAT-
- R2 pad 2: GND -> BAT-
- R3 pad 1: VCC -> VDD
- R3 pad 2: P0.06 -> Net-(Q2-Pad3)
- R5 pad 2: GND -> BAT-
- R9 pad 2: GND -> BAT-
- S1 pad 1: GND -> BAT-
- S10 pad 1: GND -> BAT-
- S11 pad 1: GND -> BAT-
- S12 pad 1: GND -> BAT-
- S13 pad 1: GND -> BAT-
- S14 pad 1: GND -> BAT-
- S15 pad 1: GND -> BAT-
- S16 pad 1: GND -> BAT-
- S17 pad 1: GND -> BAT-
- S2 pad 1: GND -> BAT-
- S3 pad 1: GND -> BAT-
- S4 pad 1: GND -> BAT-
- S5 pad 1: GND -> BAT-
- S6 pad 1: GND -> BAT-
- S7 pad 1: GND -> BAT-
- S8 pad 1: GND -> BAT-
- S9 pad 1: GND -> BAT-
- SW1 pad 2: VBAT -> BAT+
- U1 pad 1: S1 -> S13
- U1 pad 10: S9 -> S4
- U1 pad 12: GND -> BAT-
- U1 pad 15: S10 -> S8
- U1 pad 2: S2 -> S21
- U1 pad 21: GND -> BAT-
- U1 pad 24: GND -> BAT-
- U1 pad 3: S3 -> S20
- U1 pad 30: S22 -> S18
- U1 pad 32: S21 -> S17
- U1 pad 33: S20 -> S16
- U1 pad 34: S19 -> S12
- U1 pad 35: S18 -> S6
- U1 pad 36: S17 -> S7
- U1 pad 38: S16 -> S15
- U1 pad 4: S4 -> S10
- U1 pad 40: S15 -> S14
- U1 pad 41: S14 -> S1
- U1 pad 42: S13 -> S2
- U1 pad 43: S12 -> S3
- U1 pad 5: GND -> BAT-
- U1 pad 6: S5 -> S9
- U1 pad 7: S6 -> S22
- U1 pad 8: S7 -> S19
- U1 pad 9: S8 -> S5
- U2 pad 12: GND -> BAT-
- U2 pad 21: GND -> BAT-
- U2 pad 24: GND -> BAT-
- U2 pad 5: GND -> BAT-
- U3 pad 2: GND -> BAT-
- U3 pad 3: VBAT -> BAT+
- X1 pad 1: VDD -> DCCH
- X1 pad 2: DCCH -> VDD

Commit message: updated files
Parts:
- removed J2: USB-C, kbd:usb_type_c
- removed U2: E73-2G4M08S1C-52840, kbd:E73-2G4M08S1C-52840
- moved U1 0.64 mm to (88.5, 98.5)
Connections:
- J1 pad A5: Net-(J1-PadA5) -> CC1
- J1 pad B5: Net-(J1-PadB5) -> CC2
- R1 pad 1: Net-(J2-PadA5) -> CC1
- R2 pad 1: Net-(J2-PadB5) -> CC2

Commit message: autorouted
Parts:
- removed JP11: SWD_conn, kbd:connector_swd
- D2, Q1, Q2, Q3, U3: moved to B.Cu
- moved D2 1.57 mm to (61.8, 41.8)
- moved Q1 1.33 mm to (65.7, 41.9), turned to 270 degrees
- moved Q3 1.33 mm to (77.1, 41.9), turned to 270 degrees
- moved U3 1.33 mm to (69.5, 41.9), turned to 90 degrees
- moved Q2 1.28 mm to (73.5, 41.9), turned to 270 degrees
- moved X1 1.05 mm to (77.7, 40.4)
- moved C2 1.05 mm to (70.1, 40.5)
- moved C3 1.05 mm to (73.9, 40.5)
- moved R3 1.05 mm to (70.1, 41.8)
- moved R7 1.05 mm to (77.7, 41.9)
- moved R9 1.05 mm to (73.9, 41.8)
- moved D1 1.05 mm to (62.3, 40.5)
- moved R6 1.05 mm to (62.3, 41.8)
- moved C1 1.05 mm to (66.1, 40.5)
- moved R5 1.05 mm to (66.1, 41.9)
Connections:
- U1 pad 15: S8 -> S15
- U1 pad 17: S11 -> S14
- U1 pad 30: S18 -> S8
- U1 pad 32: S17 -> S3
- U1 pad 33: S16 -> S2
- U1 pad 34: S12 -> S1
- U1 pad 35: S6 -> S7
- U1 pad 36: S7 -> S6
- U1 pad 38: S15 -> S12
- U1 pad 40: S14 -> S11
- U1 pad 41: S1 -> S17
- U1 pad 42: S2 -> S16
- U1 pad 43: S3 -> S18
Routing:
- net BAT-: track 0.00 -> 829.0 mm, vias 0 -> 2
- net LED_VCC: track 0.00 -> 542.0 mm, vias 0 -> 17
- net /GND_B: track 0.00 -> 183.9 mm, vias 0 -> 1
- net D-: track 0.00 -> 153.9 mm, vias 0 -> 4
- net VBUS: track 0.00 -> 135.8 mm, vias 0 -> 3
- net VDD: track 0.00 -> 133.9 mm, vias 0 -> 6
- net /VCC_B: track 0.00 -> 122.8 mm, vias 0 -> 4
- net BAT+: track 0.00 -> 120.2 mm, vias 0 -> 4
- net S1: track 0.00 -> 99.1 mm, vias 0 -> 2
- net S2: track 0.00 -> 91.8 mm, vias 0 -> 3
- net RX: track 0.00 -> 89.7 mm
- net D+: track 0.00 -> 87.4 mm, vias 0 -> 2
- net VDDH: track 0.00 -> 84.0 mm, vias 0 -> 1
- net P0.06: track 0.00 -> 77.5 mm, vias 0 -> 1
- net S3: track 0.00 -> 76.7 mm, vias 0 -> 1
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