File: jorian.sch (KiCad schematic (older format))
At the start: 74 parts, among them U1 E73-2G4M08S1C-52840, U3 LP3990-3.3v

Commit message: updated
Parts:
- OLED1: footprint kbd:connector_i2c -> kbd:oled_128x32_i2c
Changed lines of the file:
@@
 F 0 "OLED1" H 14350 2050 50  0000 C CNN
 F 1 "I2C_conn" H 14350 2650 50  0000 C CNN
-F 2 "kbd:connector_i2c" H 14350 2400 50  0001 C CNN
+F 2 "kbd:oled_128x32_i2c" H 14350 2400 50  0001 C CNN
 F 3 "" H 14350 2400 50  0001 C CNN
 	1    14350 2400

Commit message: updated files
Parts:
- removed U3: LP3990-3.3v, kbd:SOT-23-5, symbol kbd:LP3990-3.3v
- added C3: 10uF, Capacitor_SMD:C_0805_2012Metric, symbol Device:C
- added D1: CHG, LED_SMD:LED_0603_1608Metric, symbol Device:LED
- added D2: 1N5819, Diode_SMD:D_SOD-323, symbol Diode:MBR0520
- added J1, J2: MicroUSB, kbd:usb_micro_custom, symbol Connector:USB_B_Micro
- added J3, J4: USB-C, kbd:usb_type_c, symbol jorian-rescue:USB_C_Receptacle_USB2.0-Connector
- added J5: MJ-4PP-9, kbd:trrs_connector, symbol kbd:kbd_MJ-4PP-9
- added JP11: SWD_conn, kbd:connector_swd, symbol Connector_Generic:Conn_01x04
- added JP12: TX, kbd:jumper, symbol Device:Jumper_NO_Small
- added JP13: RX, kbd:jumper, symbol Device:Jumper_NO_Small
- added JP14, JP17: VCC, kbd:jumper, symbol Device:Jumper_NO_Small
- added JP15, JP22: GND, kbd:jumper, symbol Device:Jumper_NO_Small
- added JP23: D+, kbd:jumper, symbol Device:Jumper_NO_Small
- added JP24: D-, kbd:jumper, symbol Device:Jumper_NO_Small
- added Q1: AO3407, Package_TO_SOT_SMD:SOT-23, symbol Transistor_FET:BSS83P
- added R1, R2: 5.1K, Resistor_SMD:R_0603_1608Metric, symbol Device:R
- added R3, R4: 1.5K, kbd:R_0805, symbol Device:R
- added R5, R8: 100K, Resistor_SMD:R_0603_1608Metric, symbol Device:R
- added R6: 1K, Resistor_SMD:R_0603_1608Metric, symbol Device:R
- added R7: 10K, Resistor_SMD:R_0603_1608Metric, symbol Device:R
- added R9: 4.7K, Resistor_SMD:R_0603_1608Metric, symbol Device:R
- added SW1: MSK-12C02, kbd:switch_MSK-12C02_smd, symbol Switch:SW_SPDT
- added U2: MCP73831, Package_TO_SOT_SMD:SOT-23-5, symbol Battery_Management:MCP73831-2-OT
- added U3: AP2112K-3.3, Package_TO_SOT_SMD:SOT-23-5, symbol Regulator_Linear:AP2112K-3.3
- C1, C2: value 1uF -> 10uF; footprint kbd:C_0805 -> Capacitor_SMD:C_0805_2012Metric
Connections:
- net labels added: D+, D-, P0.26, RX, TX, VBAT, VBUS, VUSB
- net labels removed: OUT+, OUT-
- wire segments 252 -> 334
- no-connect marks 4 -> 15
Other:
- note added: "LiPo Charging\n"
- note added: "Power and Filtering"
- moved on the sheet: JP16, U1

Commit message: updated files
Parts:
- removed JP16: SWD_conn, kbd:connector_swd, symbol Connector_Generic:Conn_01x04
- added JP16, JP25, JP26, JP27, JP28, JP29, JP30, JP31: (no value), kbd:jumper, symbol Device:Jumper_NO_Small
- added OLED2: I2C_conn, kbd:connector_i2c, symbol Connector_Generic:Conn_01x04
- OLED1: footprint kbd:oled_128x32_i2c -> kbd:connector_i2c
Connections:
- wire segments 334 -> 356
Other:
- moved on the sheet: JP2, JP3, JP4, JP5, JP6, JP7, JP8, JP9, OLED1

Commit message: updated files
Parts:
- removed JP12: TX, kbd:jumper, symbol Device:Jumper_NO_Small
- removed JP13: RX, kbd:jumper, symbol Device:Jumper_NO_Small
- removed JP14, JP17: VCC, kbd:jumper, symbol Device:Jumper_NO_Small
- removed JP15, JP22: GND, kbd:jumper, symbol Device:Jumper_NO_Small
- removed JP23: D+, kbd:jumper, symbol Device:Jumper_NO_Small
- removed JP24: D-, kbd:jumper, symbol Device:Jumper_NO_Small
- removed R3, R4: 1.5K, kbd:R_0805, symbol Device:R
- C1, C2, C3: footprint Capacitor_SMD:C_0805_2012Metric -> Capacitor_SMD:C_0603_1608Metric
- D2: footprint Diode_SMD:D_SOD-323 -> Diode_SMD:D_SOD-123
Connections:
- net labels removed: TX
- wire segments 356 -> 327
- no-connect marks 15 -> 16

Commit message: updated files
Parts:
- added U4: E73-2G4M08S1C-52840, kbd:E73-2G4M08S1C-52840-mod, symbol jorian-rescue:E73-2G4M08S1C-52840
- U1: footprint kbd:E73-2G4M08S1C-52840 -> kbd:E73-2G4M08S1C-52840-mod
Other:
- moved on the sheet: U1
Changed lines of the file:
@@
 L jorian-rescue:E73-2G4M08S1C-52840 U1
 U 1 1 5D9A1834
-P 2375 3075
-F 0 "U1" H 2350 4440 50  0000 C CNN
-F 1 "E73-2G4M08S1C-52840" H 2350 4349 50  0000 C CNN
-F 2 "kbd:E73-2G4M08S1C-52840" H 2375 3075 50  0001 C CNN
-F 3 "" H 2375 3075 50  0001 C CNN
-	1    2375 3075
+P 1675 2125
+F 0 "U1" H 1650 3490 50  0000 C CNN
+F 1 "E73-2G4M08S1C-52840" H 1650 3399 50  0000 C CNN
+F 2 "kbd:E73-2G4M08S1C-52840-mod" H 1675 2125 50  0001 C CNN
+F 3 "" H 1675 2125 50  0001 C CNN
+	1    1675 2125
 	1    0    0    -1
 $EndComp
@@
 $EndComp
 NoConn ~ 12375 2800
+$Comp
+L jorian-rescue:E73-2G4M08S1C-52840 U4
+U 1 1 5DDEC6CE
+P 1700 4900
+F 0 "U4" H 1675 6265 50  0000 C CNN
+F 1 "E73-2G4M08S1C-52840" H 1675 6174 50  0000 C CNN
+F 2 "kbd:E73-2G4M08S1C-52840-mod" H 1700 4900 50  0001 C CNN
+F 3 "" H 1700 4900 50  0001 C CNN
+	1    1700 4900
+	1    0    0    -1
+$EndComp
 $EndSCHEMATC

Commit message: updated files
Parts:
- J3, J4: footprint kbd:usb_type_c -> kbd:HRO-TYPE-C-31-M-12-Assembly
Changed lines of the file:
@@
 F 0 "J4" H 14355 8642 50  0000 C CNN
 F 1 "USB-C" H 14355 8551 50  0000 C CNN
-F 2 "kbd:usb_type_c" H 14400 7775 50  0001 C CNN
+F 2 "kbd:HRO-TYPE-C-31-M-12-Assembly" H 14400 7775 50  0001 C CNN
 F 3 "https://www.usb.org/sites/default/files/documents/usb_type-c.zip" H 14400 7775 50  0001 C CNN
 	1    14250 7775
@@
 F 0 "J3" H 14355 6467 50  0000 C CNN
 F 1 "USB-C" H 14355 6376 50  0000 C CNN
-F 2 "kbd:usb_type_c" H 14400 5600 50  0001 C CNN
+F 2 "kbd:HRO-TYPE-C-31-M-12-Assembly" H 14400 5600 50  0001 C CNN
 F 3 "https://www.usb.org/sites/default/files/documents/usb_type-c.zip" H 14400 5600 50  0001 C CNN
 	1    14250 5600

Commit message: updated files
Parts:
- removed R8: 100K, Resistor_SMD:R_0603_1608Metric, symbol Device:R
- removed U3: AP2112K-3.3, Package_TO_SOT_SMD:SOT-23-5, symbol Regulator_Linear:AP2112K-3.3
- added X1: 10uH, Inductor_SMD:L_0603_1608Metric, symbol pspice:INDUCTOR
- J1: renamed from J4; footprint kbd:HRO-TYPE-C-31-M-12-Assembly -> kbd:usb_type_c
- J2: renamed from J3; footprint kbd:HRO-TYPE-C-31-M-12-Assembly -> kbd:usb_type_c
- U1: footprint kbd:E73-2G4M08S1C-52840-mod -> kbd:E73-2G4M08S1C-52840
- U2: renamed from U4; footprint kbd:E73-2G4M08S1C-52840-mod -> kbd:E73-2G4M08S1C-52840
- renumbered J1 to J3, J2 to J4, U2 to U3
Connections:
- net labels added: DCCH, P0.04, P0.05, P0.06, P0.07, P0.08, P0.12, PGND, POWER_PIN, RESET, SWITCH_PIN, VDD, VDDH
- wire segments 327 -> 334
Other:
- note added: "underside pins"
- moved on the sheet: C3, J1, J2, J3, J4, J5, R1, R2

Commit message: updated files
Parts:
- OLED1: footprint kbd:connector_i2c -> kbd:connector_swd
Connections:
- no-connect marks 16 -> 18
Changed lines of the file:
@@
 	1    0    0    -1
 $EndComp
+Text Label 10750 8200 0    50   ~ 0
+GND
+Text Label 10750 8300 0    50   ~ 0
+S18
 Text Label 10750 8000 0    50   ~ 0
-GND
-Text Label 10750 8100 0    50   ~ 0
-S18
-Text Label 10750 8300 0    50   ~ 0
 VCC
 $Comp
@@
 	1    0    0    -1
 $EndComp
-Text Label 9900 5150 2    50   ~ 0
-GND
-Text Label 9900 5250 2    50   ~ 0
+Text Label 9900 5450 2    50   ~ 0
 S19
-Text Label 9900 5350 2    50   ~ 0
+Text Label 9900 6150 2    50   ~ 0
 S20
-Text Label 9900 6650 2    50   ~ 0
-S21
 $Comp
 L Connector_Generic:Conn_01x04 E21
@@
 	1    0    0    -1
 $EndComp
-Text Label 9900 6550 2    50   ~ 0
-GND
 Text Label 9900 5950 2    50   ~ 0
 S22
-Text Label 9900 6850 2    50   ~ 0
-VCC
-Text Label 10750 8200 0    50   ~ 0
+Text Label 10750 8100 0    50   ~ 0
 DIN18
+Text Label 10150 8300 2    50   ~ 0
+S18_A
+Text Label 10150 8200 2    50   ~ 0
+GND_A
+Text Label 10150 8000 2    50   ~ 0
+VCC_A
 Text Label 10150 8100 2    50   ~ 0
-S18_A
-Text Label 10150 8000 2    50   ~ 0
-GND_A
-Text Label 10150 8300 2    50   ~ 0
-VCC_A
-Text Label 10150 8200 2    50   ~ 0
 DIN18_A
-Text Label 10500 5150 0    50   ~ 0
-GND_B
-Text Label 10500 5250 0    50   ~ 0
+Text Label 10500 5450 0    50   ~ 0
 S19_B
-Text Label 10500 5350 0    50   ~ 0
+Text Label 10500 6150 0    50   ~ 0
 S20_B
-Text Label 10500 6650 0    50   ~ 0
+Text Label 10500 6850 0    50   ~ 0
 S21_B
-Text Label 10500 6550 0    50   ~ 0
-GND_B
 Text Label 10500 5950 0    50   ~ 0
 S22_B
-Text Label 10500 6850 0    50   ~ 0
+Text Label 10500 6650 0    50   ~ 0
 VCC_B
-Text Label 10500 6750 0    50   ~ 0
+Text Label 10500 5250 0    50   ~ 0
 DIN21_B
-Text Label 9900 5450 2    50   ~ 0
+Text Label 9900 5150 2    50   ~ 0
 DIN5
-Text Label 10500 5450 0    50   ~ 0
+Text Label 10500 5150 0    50   ~ 0
 DIN5_B
-Text Label 9900 6750 2    50   ~ 0
+Text Label 9900 5250 2    50   ~ 0
 DIN21
 $Comp
@@
 	1    0    0    -1
 $EndComp
-Text Label 9900 5850 2    50   ~ 0
-GND
-Text Label 10500 5850 0    50   ~ 0
-GND_B
 Wire Wire Line
 	4700 1750 4700 2350
@@
 	1    0    0    -1
 $EndComp
-NoConn ~ 10500 6050
-NoConn ~ 9900 6050
-Text Label 9900 6150 2    50   ~ 0
-VCC
-Text Label 10500 6150 0    50   ~ 0
-VCC_B
 $Comp
 L Connector_Generic:Conn_01x04 OLED1
@@
 F 0 "OLED1" H 14675 1325 50  0000 C CNN
 F 1 "I2C_conn" H 14675 1925 50  0000 C CNN
-F 2 "kbd:connector_i2c" H 14675 1675 50  0001 C CNN
+F 2 "kbd:connector_swd" H 14675 1675 50  0001 C CNN
 F 3 "" H 14675 1675 50  0001 C CNN
 	1    14675 1675
@@
 Text GLabel 2325 2625 2    50   Input ~ 0
 RX
+Text Label 9900 6750 2    50   ~ 0
+GND
+Text Label 10500 6750 0    50   ~ 0
+GND_B
+Text Label 9900 6050 2    50   ~ 0
+GND
+Text Label 9900 6650 2    50   ~ 0
+VCC
+Text Label 9900 6850 2    50   ~ 0
+S21
+Text Label 9900 5350 2    50   ~ 0
+GND
+Text Label 10500 5350 0    50   ~ 0
+GND_B
+NoConn ~ 10500 6550
+NoConn ~ 9900 6550
+NoConn ~ 9900 5850
+NoConn ~ 10500 5850
+Text Label 10500 6050 0    50   ~ 0
+GND_B
 $EndSCHEMATC
